Commit message: Modifications to support t265 + d435

File: realsense2_description/urdf/_d435.urdf.xacro (robot description, xacro)
@@ -37,13 +37,13 @@
     <xacro:property name="d435_cam_depth_pz" value="${d435_cam_height/2}"/>
     <!-- camera body, with origin at bottom screw mount -->
-    <joint name="${name}_joint" type="fixed">
+    <!--joint name="${name}_joint" type="fixed">
       <xacro:insert_block name="origin" />
       <parent link="${parent}"/>
       <child link="${name}_bottom_screw_frame" />
     </joint>
-    <link name="${name}_bottom_screw_frame"/>
+    <link name="${name}_bottom_screw_frame"/-->
     <joint name="${name}_link_joint" type="fixed">
-      <origin xyz="${d435_mesh_x_offset} ${d435_cam_depth_py} ${d435_cam_depth_pz}" rpy="0 0 0"/>
-      <parent link="${name}_bottom_screw_frame"/>
+      <xacro:insert_block name="origin" />
+      <parent link="${parent}"/>
       <child link="${name}_link" />
     </joint>

File: realsense2_description/urdf/test_d435_camera.urdf.xacro (robot description, xacro)
@@ -3,7 +3,7 @@
   <xacro:arg name="use_nominal_extrinsics" default="false"/>
   <xacro:include filename="$(find realsense2_description)/urdf/_d435.urdf.xacro" />
-  <link name="base_link" />
-  <xacro:sensor_d435 parent="base_link" use_nominal_extrinsics="$(arg use_nominal_extrinsics)">
-    <origin xyz="0 0 0" rpy="0 0 0"/>
+  <link name="t265_link" />
+  <xacro:sensor_d435 parent="t265_link" name="d435i" use_nominal_extrinsics="$(arg use_nominal_extrinsics)">
+    <origin xyz="0 0.021 0.027" rpy="0 0 0"/>
   </xacro:sensor_d435>
 </robot>
